Commit message: design is successfully imported

File: model/robot_arm_urdf.xacro (robot description, xacro)
@@ -27,19 +27,19 @@
       <geometry>
         <mesh
-          filename="file://$(find robot_arm_description)/model/meshes/base_link.STL" />
-      </geometry>
-      <material
-        name="">
-        <color
-          rgba="0.79216 0.81961 0.93333 1" />
-      </material>
-    </visual>
-    <collision>
-      <origin
-        xyz="0 0 0"
-        rpy="0 0 0" />
-      <geometry>
-        <mesh
-          filename="file://$(find robot_arm_description)/model/meshes/base_link.STL" />
+          filename="file://$(find robot_fd)/model/meshes/base_link.STL" />
+      </geometry>
+      <material
+        name="">
+        <color
+          rgba="0.79216 0.81961 0.93333 1" />
+      </material>
+    </visual>
+    <collision>
+      <origin
+        xyz="0 0 0"
+        rpy="0 0 0" />
+      <geometry>
+        <mesh
+          filename="file://$(find robot_fd)/model/meshes/base_link.STL" />
       </geometry>
     </collision>
@@ -67,5 +67,5 @@
       <geometry>
         <mesh
-          filename="file://$(find robot_arm_description)/model/meshes/link_1.STL" />
+          filename="file://$(find robot_fd)/model/meshes/link_1.STL" />
       </geometry>
       <material
@@ -81,5 +81,5 @@
       <geometry>
         <mesh
-          filename="file://$(find robot_arm_description)/model/meshes/link_1.STL" />
+          filename="file://$(find robot_fd)/model/meshes/link_1.STL" />
       </geometry>
     </collision>
@@ -125,19 +125,19 @@
       <geometry>
         <mesh
-          filename="file://$(find robot_arm_description)/model/meshes/link_2.STL" />
-      </geometry>
-      <material
-        name="">
-        <color
-          rgba="0.79216 0.81961 0.93333 1" />
-      </material>
-    </visual>
-    <collision>
-      <origin
-        xyz="0 0 0"
-        rpy="0 0 0" />
-      <geometry>
-        <mesh
-          filename="file://$(find robot_arm_description)/model/meshes/link_2.STL" />
+          filename="file://$(find robot_fd)/model/meshes/link_2.STL" />
+      </geometry>
+      <material
+        name="">
+        <color
+          rgba="0.79216 0.81961 0.93333 1" />
+      </material>
+    </visual>
+    <collision>
+      <origin
+        xyz="0 0 0"
+        rpy="0 0 0" />
+      <geometry>
+        <mesh
+          filename="file://$(find robot_fd)/model/meshes/link_2.STL" />
       </geometry>
     </collision>
@@ -183,19 +183,19 @@
       <geometry>
         <mesh
-          filename="file://$(find robot_arm_description)/model/meshes/link_3.STL" />
-      </geometry>
-      <material
-        name="">
-        <color
-          rgba="0.79216 0.81961 0.93333 1" />
-      </material>
-    </visual>
-    <collision>
-      <origin
-        xyz="0 0 0"
-        rpy="0 0 0" />
-      <geometry>
-        <mesh
-          filename="file://$(find robot_arm_description)/model/meshes/link_3.STL" />
+          filename="file://$(find robot_fd)/model/meshes/link_3.STL" />
+      </geometry>
+      <material
+        name="">
+        <color
+          rgba="0.79216 0.81961 0.93333 1" />
+      </material>
+    </visual>
+    <collision>
+      <origin
+        xyz="0 0 0"
+        rpy="0 0 0" />
+      <geometry>
+        <mesh
+          filename="file://$(find robot_fd)/model/meshes/link_3.STL" />
       </geometry>
     </collision>
@@ -241,19 +241,19 @@
       <geometry>
         <mesh
-          filename="file://$(find robot_arm_description)/model/meshes/link_4.STL" />
-      </geometry>
-      <material
-        name="">
-        <color
-          rgba="0.79216 0.81961 0.93333 1" />
-      </material>
-    </visual>
-    <collision>
-      <origin
-        xyz="0 0 0"
-        rpy="0 0 0" />
-      <geometry>
-        <mesh
-          filename="file://$(find robot_arm_description)/model/meshes/link_4.STL" />
+          filename="file://$(find robot_fd)/model/meshes/link_4.STL" />
+      </geometry>
+      <material
+        name="">
+        <color
+          rgba="0.79216 0.81961 0.93333 1" />
+      </material>
+    </visual>
+    <collision>
+      <origin
+        xyz="0 0 0"
+        rpy="0 0 0" />
+      <geometry>
+        <mesh
+          filename="file://$(find robot_fd)/model/meshes/link_4.STL" />
       </geometry>
     </collision>
@@ -299,19 +299,19 @@
       <geometry>
         <mesh
-          filename="file://$(find robot_arm_description)/model/meshes/link_5.STL" />
-      </geometry>
-      <material
-        name="">
-        <color
-          rgba="0.79216 0.81961 0.93333 1" />
-      </material>
-    </visual>
-    <collision>
-      <origin
-        xyz="0 0 0"
-        rpy="0 0 0" />
-      <geometry>
-        <mesh
-          filename="file://$(find robot_arm_description)/model/meshes/link_5.STL" />
+          filename="file://$(find robot_fd)/model/meshes/link_5.STL" />
+      </geometry>
+      <material
+        name="">
+        <color
+          rgba="0.79216 0.81961 0.93333 1" />
+      </material>
+    </visual>
+    <collision>
+      <origin
+        xyz="0 0 0"
+        rpy="0 0 0" />
+      <geometry>
+        <mesh
+          filename="file://$(find robot_fd)/model/meshes/link_5.STL" />
       </geometry>
     </collision>
@@ -357,19 +357,19 @@
       <geometry>
         <mesh
-          filename="file://$(find robot_arm_description)/model/meshes/link_6.STL" />
-      </geometry>
-      <material
-        name="">
-        <color
-          rgba="0.79216 0.81961 0.93333 1" />
-      </material>
-    </visual>
-    <collision>
-      <origin
-        xyz="0 0 0"
-        rpy="0 0 0" />
-      <geometry>
-        <mesh
-          filename="file://$(find robot_arm_description)/model/meshes/link_6.STL" />
+          filename="file://$(find robot_fd)/model/meshes/link_6.STL" />
+      </geometry>
+      <material
+        name="">
+        <color
+          rgba="0.79216 0.81961 0.93333 1" />
+      </material>
+    </visual>
+    <collision>
+      <origin
+        xyz="0 0 0"
+        rpy="0 0 0" />
+      <geometry>
+        <mesh
+          filename="file://$(find robot_fd)/model/meshes/link_6.STL" />
       </geometry>
     </collision>
@@ -415,19 +415,19 @@
       <geometry>
         <mesh
-          filename="file://$(find robot_arm_description)/model/meshes/link_7.STL" />
-      </geometry>
-      <material
-        name="">
-        <color
-          rgba="0.79216 0.81961 0.93333 1" />
-      </material>
-    </visual>
-    <collision>
-      <origin
-        xyz="0 0 0"
-        rpy="0 0 0" />
-      <geometry>
-        <mesh
-          filename="file://$(find robot_arm_description)/model/meshes/link_7.STL" />
+          filename="file://$(find robot_fd)/model/meshes/link_7.STL" />
+      </geometry>
+      <material
+        name="">
+        <color
+          rgba="0.79216 0.81961 0.93333 1" />
+      </material>
+    </visual>
+    <collision>
+      <origin
+        xyz="0 0 0"
+        rpy="0 0 0" />
+      <geometry>
+        <mesh
+          filename="file://$(find robot_fd)/model/meshes/link_7.STL" />
       </geometry>
     </collision>

Commit message: robot root link is created to fix it to the graound.

File: model/robot_arm_urdf.xacro (robot description, xacro)
@@ -6,4 +6,10 @@
   name="robot_arm_urdf" xmlns:xacro="http://www.ros.org/wiki/xacro">
   <xacro:include filename="ros2_control.xacro" />
+  <link name="world" />
+  <joint name="fixed_base_joint" type="fixed">
+    <parent link="world" />
+    <child link="base_link" />
+    <origin xyz="0 0 0" rpy="0 0 0" />
+  </joint>
   <link
     name="base_link">

Commit message: now the project includes joint 6 with mimic.

File: model/robot_arm_urdf.xacro (robot description, xacro)
@@ -457,4 +457,7 @@
       effort="100"
       velocity="3" />
+    <mimic
+      joint="joint_6"
+      multiplier="-1" />
   </joint>
 </robot>

File: model/ros2_control.xacro (robot description, xacro)
@@ -37,6 +37,14 @@
       </joint>
     </xacro:macro>
+    <xacro:macro name="gripper_mimic_joint" params="name">
+      <joint name="${name}">
+        <state_interface name="position">
+          <param name="initial_value">0.0</param>
+        </state_interface>
+        <state_interface name="velocity"/>
+      </joint>
+    </xacro:macro>
     <xacro:gripper_joint name="joint_6"/>
-    <xacro:gripper_joint name="joint_7"/>
+    <xacro:gripper_mimic_joint name="joint_7"/>
   </ros2_control>
   <!-- Gazebo system plugin -->
